File: Wave.kicad_pcb (KiCad board)
At the start: 4 copper layers, 88.1 x 80 mm, 234 parts, among them J1 USB_C_Receptacle_USB2.0_16P, J2 4 Ohm SPEAKER, J3 Conn_01x02, J4 PJ-342 / PJ-393-A, Q1 AO3400A, Q2 AO3400A, SW1 SW_Push, SW2 SW_Push, SW3 SW_Push, SW4 SW_Push, SW5 SW_Push, SW6 SW_Push, SW7 SW_Push, SW8 SW_Push, U1 SRV05-4, U10 74LVC1G08, U11 ZL38063, U12 W25Q16JVSS, U13 SN74LVC1G126DBV, U14 VEML7700-TR, U2 NS4150, U4 SN74LVC1G126DBV, U5 ESP32-S3-WROOM-1, U8 74LVC1G17, U9 SN74LVC2G74, Y1 12MHz

Commit message: Added DSP, Neopixles, MIC's and mounting holes
Parts:
- removed J4: PJ-342 / PJ-393-A, Connector_Audio:Jack_3.5mm_PJ311_Horizontal
- added C76: 0.1uF/10V(10%), Capacitor_SMD:C_0402_1005Metric, F.Cu at (115.9, 75.0)
- added C77: 0.1uF/10V(10%), Capacitor_SMD:C_0402_1005Metric, F.Cu at (115.9, 77.0)
- added C78: 0.1uF/10V(10%), Capacitor_SMD:C_0402_1005Metric, F.Cu at (115.9, 79.0)
- added H1: MountingHole_Pad, MountingHole:MountingHole_3.2mm_M3_Pad_Via, F.Cu at (27.5, 39.9)
- added H2: MountingHole_Pad, MountingHole:MountingHole_3.2mm_M3_Pad_Via, F.Cu at (85.5, 39.9)
- added H3: MountingHole_Pad, MountingHole:MountingHole_3.2mm_M3_Pad_Via, F.Cu at (90.5, 85.9)
- added H4: MountingHole_Pad, MountingHole:MountingHole_3.2mm_M3_Pad_Via, F.Cu at (22.5, 85.9)
- added MK1: ZTS6577, Knowles_LGA-5_3.5x2.65mm:Knowles_LGA-5_3.5x2.65mm, F.Cu at (56.5, 108.0)
- added MK2: ZTS6577, Knowles_LGA-5_3.5x2.65mm:Knowles_LGA-5_3.5x2.65mm, F.Cu at (20.1, 45.0)
- added MK3: ZTS6577, Knowles_LGA-5_3.5x2.65mm:Knowles_LGA-5_3.5x2.65mm, F.Cu at (92.9, 45.0)
- added R23: 33R(5%), Resistor_SMD:R_0402_1005Metric, F.Cu at (110.1, 75.0)
- added R79: 10K(5%), Resistor_SMD:R_0402_1005Metric, F.Cu at (110.1, 79.0)
- added R80: 33R(5%), Resistor_SMD:R_0402_1005Metric, F.Cu at (110.1, 81.0)
- added R81: 33R(5%), Resistor_SMD:R_0402_1005Metric, F.Cu at (110.1, 83.0)
- added R82: 10K(5%), Resistor_SMD:R_0402_1005Metric, F.Cu at (110.1, 85.0)
- added R83: 33R(5%), Resistor_SMD:R_0402_1005Metric, F.Cu at (113.0, 75.0)
- added R84: 33R(5%), Resistor_SMD:R_0402_1005Metric, F.Cu at (113.0, 77.0)
- added R85: 10K(5%), Resistor_SMD:R_0402_1005Metric, F.Cu at (113.0, 79.0)
- added R86: 33R(5%), Resistor_SMD:R_0402_1005Metric, F.Cu at (113.0, 81.0)
- added R87: 33R(5%), Resistor_SMD:R_0402_1005Metric, F.Cu at (113.0, 83.0)
- C1, C10, C11, C12, C13, C14, C15, C17, C2, C20, C21, C22, C23, C24, C25, C26, C27, C28, C29, C3, C30, C31, C32, C33, C34, C36, C37, C38, C39, C4, C40, C42, C43, C45, C46, C47, C48, C49, C5, C50, C51, C52, C53, C54, C55, C56, C57, C58, C59, C6, C60, C61, C62, C63, C68, C69, C7, C70, C71, C72, C73, C74, C75, C8, C9: footprint Capacitor_SMD:C_0603_1608Metric -> Capacitor_SMD:C_0402_1005Metric
- C16: value 0.1uF/16v(10%) -> 0.1uF/10V(10%); footprint Capacitor_SMD:C_0603_1608Metric -> Capacitor_SMD:C_0402_1005Metric
- C18: value 1uF/10V(20%) -> 1uF/10V(10%); footprint Capacitor_SMD:C_0603_1608Metric -> Capacitor_SMD:C_0402_1005Metric
- C19: value 1uF/10v(20%) -> 1uF/10v(10%); footprint Capacitor_SMD:C_0603_1608Metric -> Capacitor_SMD:C_0402_1005Metric
- C35, C41: value 1uF/16V(10%) -> 1uF/10V(10%); footprint Capacitor_SMD:C_0603_1608Metric -> Capacitor_SMD:C_0402_1005Metric
- C44: value 0.1uF/50V(10%) -> 0.1uF/10V(10%); footprint Capacitor_SMD:C_0603_1608Metric -> Capacitor_SMD:C_0402_1005Metric
- C64, C65, C66, C67: value 1uF/25V(10%) -> 1uF/10V(10%); footprint Capacitor_SMD:C_0603_1608Metric -> Capacitor_SMD:C_0402_1005Metric
- R1, R10, R11, R12, R13, R14, R15, R16, R17, R18, R19, R2, R20, R21, R22, R24, R25, R26, R27, R28, R29, R3, R30, R31, R32, R33, R34, R35, R36, R37, R38, R39, R4, R40, R41, R42, R43, R44, R45, R46, R47, R48, R49, R5, R50, R51, R52, R53, R54, R55, R56, R57, R58, R59, R6, R60, R61, R62, R63, R64, R65, R66, R67, R68, R69, R7, R70, R71, R72, R74, R75, R76, R77, R78, R8, R9: footprint Resistor_SMD:R_0603_1608Metric -> Resistor_SMD:R_0402_1005Metric
- R73: value 10K(1%) -> 33R(5%); footprint Resistor_SMD:R_0603_1608Metric -> Resistor_SMD:R_0402_1005Metric
- TP1, TP10, TP11, TP12, TP13, TP14, TP15, TP16, TP17, TP18, TP19, TP2, TP20, TP21, TP22, TP23, TP24, TP25, TP26, TP27, TP28, TP29, TP3, TP4, TP5, TP6, TP7, TP8, TP9: footprint TestPoint:TestPoint_Pad_D1.5mm -> TestPoint:TestPoint_Pad_D1.0mm
- U12: footprint Package_SO:SOIC-8_5.23x5.23mm_P1.27mm -> Package_SO:SOIC-8_3.9x4.9mm_P1.27mm
- Y1: footprint Crystal:Crystal_SMD_7050-4Pin_7.0x5.0mm -> Crystal:Crystal_SMD_2520-4Pin_2.5x2.0mm
- moved R64 137.8 mm to (53.0, 67.4), turned to 180 degrees
- moved R65 137.5 mm to (53.0, 68.4), turned to 180 degrees
- moved R66 137.1 mm to (53.0, 69.4), turned to 180 degrees
- moved R67 136.8 mm to (53.0, 70.4), turned to 180 degrees
- moved R68 136.5 mm to (53.0, 71.4), turned to 180 degrees
- moved R70 134.4 mm to (54.5, 73.0), turned to -90 degrees
- moved R69 133.8 mm to (55.5, 72.9), turned to -90 degrees
- moved Y1 132.6 mm to (61.8, 57.3), turned to 90 degrees
- moved TP22 132.1 mm to (48.6, 71.4)
- moved R56 130.6 mm to (53.0, 59.4), turned to 180 degrees
- moved R57 130.5 mm to (53.0, 60.4), turned to 180 degrees
- moved R58 130.3 mm to (53.0, 61.4), turned to 180 degrees
- moved TP21 130.2 mm to (50.6, 70.4)
- moved R59 130.2 mm to (53.0, 62.4), turned to 180 degrees
- moved R60 130.1 mm to (53.0, 63.4), turned to 180 degrees
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Connections:
- R73 pad 1: Aud_VDD -> unconnected-(R73-Pad1)
- R73 pad 2: MUTE_DATA -> unconnected-(R73-Pad2)
Routing:
- removed copper zone on F.Cu, net GNDA
