File: mk-0/KiCAD/TopBoard/Interface.kicad_sch (KiCad schematic)
At the start: 65 parts, among them Q1 AO3400A, SW1 SW_Push, SW2 SW_Push, SW3 SW_Push, SW4 SW_Push, U1 SN74LVC1G126DBV, U2 74LVC1G17, U3 SN74LVC2G74, U4 74AHCT1G125, U7 SN74LVC1G126DBV

Commit message: Cleanup and naming of Touchpoints
Parts:
- SW1: value SW_Push -> MUTE
- SW2: value SW_Push -> BUTTON 1
- SW3: value SW_Push -> BUTTON 2
- SW4: value SW_Push -> BUTTON 3
Other:
- moved on the sheet: C3, C40, C41, C42, D1, JP10, JP11, MK1, MK2, MK3, Q1, R39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
